File: pcb/mobo/mobo.kicad_pcb (KiCad board)
At the start: 2 copper layers, 51.6 x 89 mm, 74 parts, among them J1 SWD_10, J2 PEEL_MOTOR, J3 DRIVE_MOTOR, J4 SW1, J5 SPRING_FINGERS, J6 SW2, J7 SW1, J8 USART1, J9 SWD_10, U1 STM32F031C6Tx, U2 STM32F031K6Ux, U4 AP1117-33, U5 MC34063AD, U6 MAX3078E, U7 DRV8837, U8 DRV8837, Y1 8MHz

Commit message: Add REV12CD U1-only motherboard and three-board panel
Remove alternate U2 and its unused trace branches, retain U1 wiring, and label the derivative REV12CD. Add an editable routed three-up KiCad panel, shared PCB/stencil upload ZIP, assembly coordinates, reproducible export tools and validation reports.
Parts:
- removed G***: LOGO, index:goblin
- removed G*** (x2): LOGO, LOGO
- removed G***: pulsar, feeder:pulsar
- removed G***: LOGO, index:logo_mask
- removed U2: STM32F031K6Ux, Package_DFN_QFN:QFN-32-1EP_5x5mm_P0.5mm_EP3.45x3.45mm
- renumbered REF** to GFX1
Routing:
- net LED_B: track 48.5 -> 45.2 mm
- net PA1: track 3.26 -> 0.00 mm
- net PA3: track 3.10 -> 0.00 mm
- net MOTOR_ENABLE: track 47.2 -> 44.2 mm
- net +3V3: track 271.6 -> 269.2 mm
- net PA0: track 3.24 -> 0.82 mm
- net SW1: track 46.6 -> 44.2 mm
- net LED_G: track 48.6 -> 46.3 mm
- net LED_R: track 48.7 -> 46.4 mm
- net SWCLK: track 50.8 -> 48.8 mm
- net OSC_OUT: track 8.72 -> 6.79 mm
- net OSC_IN: track 11.3 -> 9.37 mm
- net RESET: track 54.9 -> 53.0 mm
- net ~{RE}: track 45.1 -> 43.9 mm
- net SWDIO: track 52.5 -> 51.3 mm
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Other:
- board text added: "Feeder REV12CD crazydart"
- board text removed: "LumenPnP Feeder REV12 <<hash>> Opulo Inc."

Commit message: Brand REV12CD single board with AI Herding Cats artwork
Add back logo, serial write-in area, website and repository URL in the installed orientation. Credit Opulo's original open-source design and retain the vector artwork and previews.
Other:
- board text added: "AI Herding Cats"
- board text added: "Feeder REV12CD"
- board text added: "Feeder REV12CD AI Herding Cats"
- board text added: "Original design: Opulo Open-source hardware"
- board text added: "SN:"
- board text added: "aiherdingcats.com"
- board text added: "github.com/crazydart/feeder"
- board text removed: "Feeder REV12CD crazydart"
