File: pcb/mobo-panel3/feeder-rev12cd-panel3.kicad_pcb (KiCad board)
At the start: 2 copper layers, 184 x 104 mm, 205 parts, among them P1_C1 15p, P1_C10 4.7uF, P1_C11 4.7uF, P1_C12 100uF, P1_C13 10u, P1_C14 470pF, P1_C16 470uF, P1_C17 100n, P1_C18 100n, P1_C19 100n, P1_C2 15p, P1_C20 100n, P1_C3 100n, P1_C4 100n, P1_C5 100n, P1_C6 15pF, P1_C7 100n, P1_C8 4.7uF, P1_C9 10u, P1_D1 LED_RGBA, P1_D2 SM712_SOT23, P1_D3 LED_RGBA_ALT, P1_D6 1N5819, P1_D9 MMSZ4684T1G, P1_FID1 Fiducial, P1_FID2 Fiducial, P1_FID3 Fiducial, P1_GFX1 OSHW-Symbol_6.7x6mm_Mask, P1_J1 SWD_10, P1_J2 PEEL_MOTOR, P1_J3 DRIVE_MOTOR, P1_J4 SW1, P1_J5 SPRING_FINGERS, P1_J6 SW2, P1_J7 SW1, P1_J8 USART1, P1_J9 SWD_10, P1_L1 220uH, P1_R1 1k, P1_R13 0.33R, P1_R14 220R, P1_R15 20R, P1_R16 20R, P1_R17 10K, P1_R18 1M, P1_R19 1M, P1_R2 470, P1_R3 470, P1_R4 10K, P1_R5 470, P1_R6 5.6k, P1_R7 10K, P1_R9 39k, P1_TP1 TP_3V3, P1_TP2 TP_10V, P1_TP3 TP_DRIVE_M1, P1_TP4 TP_DRIVE_M2, P1_TP5 TP_PEEL_M2, P1_TP6 TP_PEEL_M1, P1_TP7 TP_QUAD_A, P1_TP8 TP_QUAD_B, P1_U1 STM32F031C6Tx, P1_U4 AP1117-33, P1_U5 MC34063AD, P1_U6 MAX3078E, P1_U7 DRV8837, P1_U8 DRV8837, P1_Y1 8MHz, P2_C1 15p, P2_C10 4.7uF, P2_C11 4.7uF, P2_C12 100uF, P2_C13 10u, P2_C14 470pF, P2_C16 470uF, P2_C17 100n, P2_C18 100n, P2_C19 100n, P2_C2 15p, P2_C20 100n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

Commit message: Regenerate branded three-board REV12CD panel and fabrication ZIP
Copy the approved artwork and editable logo groups to all three boards. Refresh PCB and stencil Gerbers, the combined JLCPCB upload ZIP, placement handoff, previews and checksums. Verify the artwork against the source and confirm that all non-silkscreen fabrication data and existing DRC findings are unchanged.
Other:
- board text added: "AI Herding Cats"
- board text added: "Feeder REV12CD"
- board text added: "Feeder REV12CD AI Herding Cats"
- board text added: "Original design: Opulo Open-source hardware"
- board text added: "SN:"
- board text added: "aiherdingcats.com"
- board text added: "github.com/crazydart/feeder"
- board text removed: "Feeder REV12CD crazydart"
